File: fhc-pcb/fhc-pcb.kicad_pcb (KiCad board)
At the start: 2 copper layers, 16 parts, among them J1 Screw_Terminal_01x02, SW1 SW_Push_Dual, SW2 SW_Push_Dual, SW3 SW_Push_Dual, SW4 SW_Push_Dual, SW5 SW_Push_Dual, U1 WeMos_D1_mini

Commit message: First complete draft of PCB
Optimization still needed
Parts:
- moved R7 64.9 mm to (444.5, 241.3), turned to 270 degrees
- moved R4 56.4 mm to (469.9, 251.5), turned to 90 degrees
- moved SW3 56.4 mm to (476.2, 223.5)
- moved R3 50.6 mm to (469.9, 231.1), turned to 90 degrees
- moved D2 49.5 mm to (430.5, 246.4)
- moved R6 47.7 mm to (444.5, 210.8), turned to 90 degrees
- moved J1 44.9 mm to (384.8, 248.9), turned to 0 degrees
- moved U1 39.5 mm to (403.9, 208.3), turned to 270 degrees
- moved D1 36.9 mm to (430.5, 205.7)
- moved R1 34.9 mm to (469.9, 210.8), turned to 90 degrees
- moved SW5 31.4 mm to (450.9, 223.5)
- moved SW1 30.6 mm to (450.9, 203.2)
- moved SW4 30.2 mm to (450.9, 243.8)
- moved R2 29.3 mm to (419.1, 221.0), turned to 270 degrees
- moved R5 25.7 mm to (444.5, 221.0), turned to 270 degrees
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Connections:
- J1 pad 1: GND -> +5V
- J1 pad 2: +5V -> GND
- SW1 pad 1: Net-(SW1-Pad1) -> Net-(R1-Pad2)
- SW1 pad 2: Net-(R1-Pad2) -> Net-(R6-Pad1)
- SW2 pad 1: Net-(SW2-Pad1) -> Net-(R2-Pad2)
- SW2 pad 2: Net-(R2-Pad2) -> Net-(R6-Pad1)
- SW3 pad 1: Net-(SW3-Pad1) -> Net-(R3-Pad2)
- SW3 pad 2: Net-(R3-Pad2) -> Net-(R6-Pad1)
- SW4 pad 1: Net-(SW4-Pad1) -> Net-(R4-Pad2)
- SW4 pad 2: Net-(R4-Pad2) -> Net-(R6-Pad1)
- SW5 pad 1: Net-(SW5-Pad1) -> Net-(R5-Pad2)
- SW5 pad 2: Net-(R5-Pad2) -> Net-(R6-Pad1)
- U1 pad 13: Net-(SW2-Pad1) -> Net-(R2-Pad2)
- U1 pad 14: Net-(SW1-Pad1) -> Net-(R1-Pad2)
- U1 pad 4: Net-(SW3-Pad1) -> Net-(R3-Pad2)
- U1 pad 5: Net-(SW4-Pad1) -> Net-(R4-Pad2)
- U1 pad 6: Net-(SW5-Pad1) -> Net-(R5-Pad2)
Routing:
- net Net-(R6-Pad1): track 0.00 -> 209.6 mm
- net GND: track 0.00 -> 164.2 mm, vias 0 -> 2
- net Net-(R5-Pad2): track 0.00 -> 134.6 mm, vias 0 -> 1
- net Net-(R4-Pad2): track 0.00 -> 126.9 mm
- net Net-(R3-Pad2): track 0.00 -> 104.1 mm, vias 0 -> 2
- net Net-(R1-Pad2): track 0.00 -> 104.1 mm, vias 0 -> 1
- net Net-(D1-Pad1): track 0.00 -> 62.0 mm
- net Net-(D2-Pad1): track 0.00 -> 45.7 mm
- net Net-(R2-Pad2): track 0.00 -> 41.7 mm
- net +5V: track 0.00 -> 18.3 mm
- net Net-(D2-Pad2): track 0.00 -> 13.5 mm
- net Net-(D1-Pad2): track 0.00 -> 13.5 mm

Commit message: Another reroute of the PCB
Parts:
- added REF**: MountingHole_3.2mm_M3_DIN965_Pad, MountingHole:MountingHole_3.2mm_M3_DIN965_Pad, F.Cu at (100.3, 68.6)
- added REF**: MountingHole_3.2mm_M3_DIN965_Pad, MountingHole:MountingHole_3.2mm_M3_DIN965_Pad, F.Cu at (223.5, 68.6)
- added REF**: MountingHole_3.2mm_M3_DIN965_Pad, MountingHole:MountingHole_3.2mm_M3_DIN965_Pad, F.Cu at (223.5, 121.9)
- added REF**: MountingHole_3.2mm_M3_DIN965_Pad, MountingHole:MountingHole_3.2mm_M3_DIN965_Pad, F.Cu at (100.3, 121.9)
- moved J1 326.9 mm to (99.1, 90.2), turned to 270 degrees
- moved U1 307.8 mm to (118.1, 94.0), turned to 90 degrees
- moved R2 297.1 mm to (152.4, 90.2)
- moved SW1 297.1 mm to (184.2, 72.4)
- moved SW4 297.1 mm to (184.2, 113.0)
- moved SW5 297.1 mm to (184.2, 92.7)
- moved R1 297.1 mm to (203.2, 80.0)
- moved R3 297.1 mm to (203.2, 100.3)
- moved R4 297.1 mm to (203.2, 120.7)
- moved R5 297.1 mm to (177.8, 90.2)
- moved R6 297.1 mm to (177.8, 80.0)
- moved R7 297.1 mm to (177.8, 110.5)
- moved SW2 297.1 mm to (158.8, 92.7)
- moved SW3 297.1 mm to (209.6, 92.7)
- moved D1 297.1 mm to (163.8, 74.9)
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Routing:
- net Net-(R5-Pad2): track 134.6 -> 79.1 mm, vias 1 -> 2
- net GND: track 164.2 -> 214.0 mm, vias 2 -> 0
- net Net-(R6-Pad1): track 209.6 -> 163.5 mm
- net +5V: track 18.3 -> 61.1 mm
- net Net-(R4-Pad2): track 126.9 -> 85.7 mm, vias 0 -> 1
- net Net-(R2-Pad2): track 41.7 -> 70.4 mm
- net Net-(D2-Pad1): track 45.7 -> 71.5 mm, vias 0 -> 2
- net Net-(D1-Pad1): track 62.0 -> 37.1 mm
- net Net-(R1-Pad2): track 104.1 -> 84.5 mm, vias 1 -> 0
- net Net-(R3-Pad2): track 104.1 -> 117.1 mm, vias 2 -> 0
Other:
- board outline added: 133.3 x 63.5 mm
- net class JLPCB added: clearance 0.3, trace_width 0.5, via_dia 0.8, via_drill 0.4
- board text added: "OnStep Wireless Handcontroller R1"
