File: fhc-pcb/fhc-pcb.sch (KiCad schematic (older format))
At the start: 16 parts, among them J1 Screw_Terminal_01x02, SW1 SW_Push_Dual, SW2 SW_Push_Dual, SW3 SW_Push_Dual, SW4 SW_Push_Dual, SW5 SW_Push_Dual, U1 WeMos_D1_mini

Commit message: First complete draft of PCB
Optimization still needed
Parts:
- SW1, SW2, SW3, SW4, SW5: symbol Switch:SW_Push_Dual -> Switch:SW_Push
Connections:
- wire segments 66 -> 67
Other:
- moved on the sheet: J1, R1, R2, R3, R4, R5
